File: assets/pcb/NixieTubeClock/bin-to-dec_tube-driver.sch (EAGLE design)
At the start: 9 parts, among them IC1 K155ID1, P1 DEC_OUT, P2 BIN_IN, P3 HV_IN

Commit message: updates to PCB
Parts:
- removed R1: 10k, myLibrary:RESISTOR
Connections:
- removed net N$1: P1.1, R1.1
- net +V: now also P1.1; no longer R1.2
Changed lines of the file:
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@@
 <part name="U$10" library="myLibrary" deviceset="GND" device=""/>
 <part name="W1" library="myLibrary" deviceset="WIRE" device="_7.62MM"/>
-<part name="R1" library="myLibrary" deviceset="RESISTOR" device="" value="10k"/>
 <part name="U$11" library="myLibrary" deviceset="+V" device=""/>
 </parts>
@@
 <attribute name="VALUE" x="73.66" y="53.34" size="0.8128" layer="96" align="center"/>
 </instance>
-<instance part="R1" gate="R" x="78.74" y="22.86" smashed="yes" rot="R90">
-<attribute name="NAME" x="78.74" y="20.828" size="0.8128" layer="95" rot="R90" align="center-left"/>
-<attribute name="VALUE" x="81.28" y="22.86" size="0.8128" layer="96" rot="R90" align="bottom-center"/>
-</instance>
-<instance part="U$11" gate="+V" x="78.74" y="30.48" smashed="yes"/>
+<instance part="U$11" gate="+V" x="81.28" y="15.24" smashed="yes"/>
 </instances>
 <busses>
@@
 </segment>
 <segment>
-<pinref part="R1" gate="R" pin="2"/>
+<pinref part="P1" gate="P" pin="1"/>
+<wire x1="91.44" y1="15.24" x2="81.28" y2="15.24" width="0.1524" layer="91"/>
 <pinref part="U$11" gate="+V" pin="+V"/>
 </segment>
@@
 </segment>
 </net>
-<net name="N$1" class="0">
-<segment>
-<pinref part="P1" gate="P" pin="1"/>
-<pinref part="R1" gate="R" pin="1"/>
-<wire x1="91.44" y1="15.24" x2="78.74" y2="15.24" width="0.1524" layer="91"/>
-</segment>
-</net>
