File: assets/pcb/NixieTubeClock/mainboard.brd (EAGLE design)
At the start: 71.1 x 40.6 mm, 18 parts, among them J1 POW (5V), P1 MX, P2 MXX, P3 HX, P4 HXX, P5 T1, P6 T2, P7 RTC, P8 HV_EN

Commit message: updates to PCB
Parts:
- removed P5: T1, myLibrary:XH2.54_2-PIN
- removed P6: T2, myLibrary:XH2.54_2-PIN
- removed R3, R4: >1m, myLibrary:RESISTOR_10.16MM
- moved CREATOR 35.6 mm to (25.4, 20.3), turned to 90 degrees
Connections:
- removed net N$20: MC1.4, P6.2, R4.1
- removed net N$21: MC1.5, P5.2, R3.1
- removed net R: MC1.29, R3.2, R4.2
- new net N$3: MC1.6
- new net N$4: MC1.7
- new net N$5: MC1.4
- new net N$6: MC1.5
- new net N$7: MC1.9
- new net N$8: MC1.10
- net +3V3: now also P1.6, P2.6, P3.6, P4.6
- net +5V: no longer P1.6, P2.6, P3.6, P4.6
- net ACT: no longer MC1.31
- net AHX: no longer MC1.19
- net AHXX: no longer MC1.24
- net AMX: no longer MC1.9
- net AMXX: no longer MC1.14
- net BHX: no longer MC1.20
- net BHXX: no longer MC1.25
- net BMX: no longer MC1.10
- net BMXX: no longer MC1.15
- net CHX: no longer MC1.21
- net CHXX: no longer MC1.26
- net CMX: no longer MC1.11
- net CMXX: no longer MC1.16
- net DHX: no longer MC1.22
- net DHXX: no longer MC1.27
- net DMX: no longer MC1.12
- net DMXX: no longer MC1.17
- net GND: no longer P5.1, P6.1
- net HV_EN: no longer MC1.32
- net SCL: no longer MC1.7
- net SDA: no longer MC1.6
Routing:
- net N$20: track 93.9 -> 0.00 mm, vias 2 -> 0
- net N$21: track 75.3 -> 0.00 mm, vias 1 -> 0
- net R: track 21.9 -> 0.00 mm
- net ACT: track 24.8 -> 12.3 mm
- net DHXX: track 12.0 -> 6.88 mm
- net DHX: track 6.35 -> 2.54 mm
- net CHXX: track 16.3 -> 12.5 mm
- net BHX: track 35.7 -> 31.8 mm
- net CHX: track 9.20 -> 6.66 mm
- net BHXX: track 20.6 -> 18.1 mm
- net SDA: track 62.1 -> 60.3 mm
- net AHXX: track 24.2 -> 22.4 mm
- net DMX: track 6.88 -> 5.08 mm
- net CMX: track 6.88 -> 5.08 mm
- net BMX: track 6.88 -> 5.08 mm
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Other:
- board size 71.1 x 40.6 mm -> 90.2 x 40.6 mm
