File: assets/pcb/NixieTubeClock/mainboard.sch (EAGLE design)
At the start: 18 parts, among them J1 POW (5V), P1 MX, P2 MXX, P3 HX, P4 HXX, P5 T1, P6 T2, P7 RTC, P8 HV_EN

Commit message: updates to PCB
Parts:
- removed P5: T1, myLibrary:PORT_2-PIN_XH2.54
- removed P6: T2, myLibrary:PORT_2-PIN_XH2.54
- removed R3, R4: >1m, myLibrary:RESISTOR
Connections:
- removed net N$20: MC1.GP2, P6.2, R4.1
- removed net N$21: MC1.GP3, P5.2, R3.1
- removed net R: MC1.GP22, R3.2, R4.2
- new net N$3: MC1.GP4/SDA
- new net N$4: MC1.GP5/SCL
- new net N$5: MC1.GP2
- new net N$6: MC1.GP3
- new net N$7: MC1.GP6
- new net N$8: MC1.GP7
- net +3V3: now also P1.6, P2.6, P3.6, P4.6
- net +5V: no longer P1.6, P2.6, P3.6, P4.6
- net ACT: no longer MC1.GP26/ADC0
- net AHX: no longer MC1.GP14
- net AHXX: no longer MC1.GP18
- net AMX: no longer MC1.GP6
- net AMXX: no longer MC1.GP10
- net BHX: no longer MC1.GP15
- net BHXX: no longer MC1.GP19
- net BMX: no longer MC1.GP7
- net BMXX: no longer MC1.GP11
- net CHX: no longer MC1.GP16
- net CHXX: no longer MC1.GP20
- net CMX: no longer MC1.GP8
- net CMXX: no longer MC1.GP12
- net DHX: no longer MC1.GP17
- net DHXX: no longer MC1.GP21
- net DMX: no longer MC1.GP9
- net DMXX: no longer MC1.GP13
- net GND: no longer P5.1, P6.1
- net HV_EN: no longer MC1.GP27/ADC1
- net SCL: no longer MC1.GP5/SCL
- net SDA: no longer MC1.GP4/SDA
Other:
- moved on the sheet: J1, P7
