File: assets/pcb/NixieTubeClock/nixie-tube_daughterboard.brd (EAGLE design)
At the start: 35.6 x 35.6 mm, 8 parts, among them IC1 K155ID1, P1 DEC_OUT, P2 BIN_IN, P3 HV_IN

Commit message: updates to PCB
Parts:
- removed C1: 100nf, myLibrary:CAPACITOR_UNPOLARISED_5.08MM
- removed CREATOR: Isaac, myLibrary:INFO_T
- removed IC1: K155ID1, myLibrary:16-PIN_DIP
- removed P2: BIN_IN, myLibrary:XH2.54_6-PIN
- removed P3: HV_IN, myLibrary:XH2.54_2-PIN
- removed W1: (no value), myLibrary:WIRE_7.62MM
- added R1: 10k, myLibrary:RESISTOR_10.16MM
- added TUBE: IN-14, myLibrary:NIXIE-TUBE_IN-14
- P1: value DEC_OUT -> (none)
- SCHEMATIC1: value 17-09-2023 -> 19-02-24
- moved P1 30.5 mm to (2.54, 33.0), turned to 270 degrees
- moved SCHEMATIC1 7.65 mm to (3.81, 7.62)
Connections:
- removed net +5V: C1.1, IC1.5, P2.6
- removed net A: IC1.3, P2.2
- removed net B: IC1.6, P2.3
- removed net C: IC1.7, P2.4
- removed net D: IC1.4, P2.5
- removed net GND: C1.2, IC1.12, P2.1, P3.1, W1.1, W1.2
- removed net N$16: P1.2
- removed net N$17: P1.13
- new net C1: P1.2, TUBE.C1
- new net C2: P1.13, TUBE.C2
- new net N$1: R1.1, TUBE.A
- net +V: now also R1.2; no longer P3.2
- net 0: now also TUBE.0; no longer IC1.16
- net 1: now also TUBE.1; no longer IC1.15
- net 2: now also TUBE.2; no longer IC1.8
- net 3: now also TUBE.3; no longer IC1.9
- net 4: now also TUBE.4; no longer IC1.13
- net 5: now also TUBE.5; no longer IC1.14
- net 6: now also TUBE.6; no longer IC1.11
- net 7: now also TUBE.7; no longer IC1.10
- net 8: now also TUBE.8; no longer IC1.1
- net 9: now also TUBE.9; no longer IC1.2
Routing:
- net C1: track 0.00 -> 60.5 mm
- net 0: track 15.5 -> 54.9 mm, vias 1 -> 0
- net 1: track 15.4 -> 50.2 mm
- net +V: track 23.2 -> 53.4 mm
- net C2: track 0.00 -> 24.0 mm
- net N$1: track 0.00 -> 15.9 mm
- net C: track 15.5 -> 0.00 mm
- net 4: track 21.7 -> 36.6 mm, vias 1 -> 0
- net 5: track 19.3 -> 33.2 mm
- net 8: track 13.9 -> 27.3 mm
- net D: track 11.9 -> 0.00 mm
- net B: track 11.9 -> 0.00 mm, vias 1 -> 0
- net A: track 11.9 -> 0.00 mm
- net 3: track 31.2 -> 42.0 mm
- net 2: track 33.0 -> 43.8 mm
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- removed copper zone on layer 16, net +5V
- removed copper zone on layer 1, net GND
