File: assets/pcb/nixie-tube-clock_pcb/nixie-tube-clock_mainboard.sch (EAGLE design)
At the start: 14 parts, among them J1 POW (5V), P1 MX, P2 MXX, P3 HX, P4 HXX, P7 RTC, P8 HV_EN

Commit message: cleaned up files
Parts:
- added GND: GND, myLibrary:PORT_3-PIN_XH2.54
- added JP1: (no value), myLibrary:JUMPER_2-WAY_HEADER
- added P11: CAP1188, myLibrary:PORT_13-PIN_HEADER
- added P12: (no value), myLibrary:PORT_13-PIN_HEADER
- added P5: RTC_A, myLibrary:PORT_6-PIN_HEADER
- added P6: HV_OUT, myLibrary:PORT_2-PIN_HEADER
- added P9: HV_OUT, myLibrary:PORT_4-PIN_XH2.54
- added RTC_B: RTC_B, myLibrary:PORT_4-PIN_XH2.54
- added TOUCH: TOUCH, myLibrary:PORT_3-PIN_XH2.54
- CREATOR: value Isaac -> ISAAC
- P1: value MX -> MXX
- P2: value MXX -> MX
- P3: value HX -> HXX
- P4: value HXX -> HX
- P7: value RTC -> HV_IN; device myLibrary:PORT_4-PIN_XH2.54 -> myLibrary:PORT_3-PIN_HEADER
- P8: value HV_EN -> (none); device myLibrary:PORT_3-PIN_XH2.54 -> myLibrary:PORT_1-PIN_HEADER
- SCHEMATIC1: value 19-09-2023 -> 04-05-24
Connections:
- removed net HV_EN: P8.3
- removed net N$3: MC1.GP4/SDA
- removed net N$4: MC1.GP5/SCL
- removed net N$5: MC1.GP2
- removed net N$6: MC1.GP3
- removed net N$7: MC1.GP6
- removed net N$8: MC1.GP7
- new net 32K: P5.6
- new net BUZZ: MC1.GP12
- new net C1: P12.9, TOUCH.1
- new net C2: P12.8, TOUCH.2
- new net C3: P12.7, TOUCH.3
- new net C4: P12.6
- new net C5: P12.5
- new net C6: P12.4
- new net C7: P12.3
- new net C8: P12.2
- new net HV: P6.1, P9.1, P9.2, P9.3, P9.4
- new net N$9: JP1.2, P7.3
- new net SHDN: MC1.GP14, P7.1
- new net SQW: P5.5
- net +3V3: now also P11.11, P5.2, RTC_B.3; no longer P7.2
- net +5V: now also JP1.1; no longer P8.1
- net ACT: now also MC1.GP13
- net AHX: now also MC1.GP15, P4.2; no longer P3.2
- net AHXX: now also MC1.GP19, P3.2; no longer P4.2
- net AMX: now also MC1.GP8, P2.2; no longer P1.2
- net AMXX: now also MC1.GP2, P1.2; no longer P2.2
- net BHX: now also MC1.GP16, P4.3; no longer P3.3
- net BHXX: now also MC1.GP20, P3.3; no longer P4.3
- net BMX: now also MC1.GP9, P2.3; no longer P1.3
- net BMXX: now also MC1.GP3, P1.3; no longer P2.3
- net CHX: now also MC1.GP17, P4.4; no longer P3.4
- net CHXX: now also MC1.GP21, P3.4; no longer P4.4
- net CMX: now also MC1.GP10, P2.4; no longer P1.4
- net CMXX: now also MC1.GP6, P1.4; no longer P2.4
- net DHX: now also MC1.GP18, P4.5; no longer P3.5
- net DHXX: now also MC1.GP22, P3.5; no longer P4.5
- net DMX: now also MC1.GP11, P2.5; no longer P1.5
- net DMXX: now also MC1.GP7, P1.5; no longer P2.5
- net GND: now also GND.1, GND.2, GND.3, P11.10, P5.1, P6.2, P7.2, RTC_B.4; no longer P7.1, P8.2
- net SCL: now also MC1.GP5/SCL, P11.12, P5.4, RTC_B.1; no longer P7.4
- net SDA: now also MC1.GP4/SDA, P11.13, P5.3, RTC_B.2; no longer P7.3
